Commit message: fix(sim): route ground contact through a tibia sphere and lower servo damping
The flat tibia end rolled on its rim and contact forces through the 10 g foot link made the solver jitter. The foot sphere is now a collision shape on the tibia link and the foot link is visual-only. Servo velocity gain 1.0 acted as viscous drag, so it drops to 0.3.

Co-Authored-By: Claude Sonnet 5.5 <noreply@anthropic.com>

File: assets/urdf/hexapod.urdf (robot description, URDF)
Before this commit: robot hexapod, 25 links, 24 joints
Links:
- link LF_foot: geometry visual sphere radius=0.01
- link LF_tibia_link: geometry collision cylinder length=0.12 radius=0.008; collision sphere radius=0.01
- link LM_foot: geometry visual sphere radius=0.01
- link LM_tibia_link: geometry collision cylinder length=0.12 radius=0.008; collision sphere radius=0.01
- link LR_foot: geometry visual sphere radius=0.01
- link LR_tibia_link: geometry collision cylinder length=0.12 radius=0.008; collision sphere radius=0.01
- link RF_foot: geometry visual sphere radius=0.01
- link RF_tibia_link: geometry collision cylinder length=0.12 radius=0.008; collision sphere radius=0.01
- link RM_foot: geometry visual sphere radius=0.01
- link RM_tibia_link: geometry collision cylinder length=0.12 radius=0.008; collision sphere radius=0.01
- link RR_foot: geometry visual sphere radius=0.01
- link RR_tibia_link: geometry collision cylinder length=0.12 radius=0.008; collision sphere radius=0.01
